Commit message: updated urdf and proto file to add collision bodies for mpss

File: mpss_description/urdf/machines/machine_base_description.urdf (robot description, URDF)
Before this commit: robot machine, 1 links, 0 joints
Links:
- link machine_base/base_link: mass None -> 80; geometry collision box size=0.75 0.40 0.78; visual mesh filename=package://mpss_description/meshes/mps_base/meshes/mps_base_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 scale=1.0 1.0 1.0

File: mpss_description/urdf/machines/machine_cap_description.urdf (robot description, URDF)
Before this commit: robot machine, 1 links, 0 joints
Links:
- link machine_cap/base_link: mass None -> 80; geometry collision box size=0.75 0.40 0.78; visual mesh filename=package://mpss_description/meshes/mps_cap/meshes/mps_cap_fu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 scale=1.0 1.0 1.0

File: mpss_description/urdf/machines/machine_delivery_description.urdf (robot description, URDF)
Before this commit: robot machine, 1 links, 0 joints
Links:
- link machine_delivery/base_link: mass None -> 80; geometry collision box size=0.75 0.40 0.78; visual mesh filename=package://mpss_description/meshes/mps_delivery/meshes/mps_d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 scale=1.0 1.0 1.0

File: mpss_description/urdf/machines/machine_ring_description.urdf (robot description, URDF)
Before this commit: robot machine, 1 links, 0 joints
Links:
- link machine_ring/base_link: mass None -> 80; geometry collision box size=0.75 0.40 0.78; visual mesh filename=package://mpss_description/meshes/mps_ring/meshes/mps_ring_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 scale=1.0 1.0 1.0

File: mpss_description/urdf/machines/machine_storage_description.urdf (robot description, URDF)
Before this commit: robot machine, 1 links, 0 joints
Links:
- link machine_storage/base_link: mass None -> 80; geometry collision box size=0.75 0.40 0.78; visual mesh filename=package://mpss_description/meshes/mps_storage/meshes/mps_st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 scale=1.0 1.0 1.0

Commit message: mps_description: rename mpss -> mps

File: mpss_description/urdf/machines/machine_base_description.urdf (robot description, URDF)
Before this commit: robot machine, 1 links, 0 joints
Links:
- link machine_base/base_link: geometry collision box size=0.75 0.40 0.78; visual mesh filename=package://mps_description/meshes/mps_base/meshes/mps_base_f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 scale=1.0 1.0 1.0

File: mpss_description/urdf/machines/machine_cap_description.urdf (robot description, URDF)
Before this commit: robot machine, 1 links, 0 joints
Links:
- link machine_cap/base_link: geometry collision box size=0.75 0.40 0.78; visual mesh filename=package://mps_description/meshes/mps_cap/meshes/mps_cap_ful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 scale=1.0 1.0 1.0

File: mpss_description/urdf/machines/machine_delivery_description.urdf (robot description, URDF)
Before this commit: robot machine, 1 links, 0 joints
Links:
- link machine_delivery/base_link: geometry collision box size=0.75 0.40 0.78; visual mesh filename=package://mps_description/meshes/mps_delivery/meshes/mps_de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 scale=1.0 1.0 1.0

File: mpss_description/urdf/machines/machine_ring_description.urdf (robot description, URDF)
Before this commit: robot machine, 1 links, 0 joints
Links:
- link machine_ring/base_link: geometry collision box size=0.75 0.40 0.78; visual mesh filename=package://mps_description/meshes/mps_ring/meshes/mps_ring_f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 scale=1.0 1.0 1.0

File: mpss_description/urdf/machines/machine_storage_description.urdf (robot description, URDF)
Before this commit: robot machine, 1 links, 0 joints
Links:
- link machine_storage/base_link: geometry collision box size=0.75 0.40 0.78; visual mesh filename=package://mps_description/meshes/mps_storage/meshes/mps_sto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 scale=1.0 1.0 1.0
