Commit message: project: rename robotino3 -> robotino

File: robotino3_simulation/urdf/components/robotino_body.urdf.xacro (robot description, xacro)
@@ -18,5 +18,5 @@
         <origin xyz="0.01 0 0" rpy="0 0 ${M_PI/2}"/>
         <geometry>
-          <mesh filename="package://robotino3_simulation/meshes/parts/robotino_base.dae" scale="${M_SCALE} ${M_SCALE} ${M_SCALE}"/>
+          <mesh filename="package://robotino_simulation/meshes/parts/robotino_base.dae" scale="${M_SCALE} ${M_SCALE} ${M_SCALE}"/>
         </geometry>
       </visual>

File: robotino3_simulation/urdf/components/robotino_parts.urdf.xacro (robot description, xacro)
@@ -16,5 +16,5 @@
         <origin xyz="0 0 0" rpy="0 0 0"/>
         <geometry>
-          <mesh filename="package://robotino3_simulation/meshes/parts/robotino_wheel.dae" scale="${M_SCALE} ${M_SCALE} ${M_SCALE}"/>
+          <mesh filename="package://robotino_simulation/meshes/parts/robotino_wheel.dae" scale="${M_SCALE} ${M_SCALE} ${M_SCALE}"/>
         </geometry>
       </visual>
@@ -67,5 +67,5 @@
         <origin xyz="0 0 0" rpy="0 0 0"/>
         <geometry>
-          <mesh filename="package://robotino3_simulation/meshes/parts/angle_bracket_usb_hub.dae" scale="${M_SCALE} ${M_SCALE} ${M_SCALE}"/>
+          <mesh filename="package://robotino_simulation/meshes/parts/angle_bracket_usb_hub.dae" scale="${M_SCALE} ${M_SCALE} ${M_SCALE}"/>
         </geometry>
       </visual>

File: robotino3_simulation/urdf/robots/robotino3_description.urdf (robot description, URDF)
Before this commit: robot robotino, 6 links, 5 joints
Links:
- link anglebracketusb_link: geometry visual mesh filename=package://robotino_simulation/meshes/parts/angle_bracket_us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 scale=0.01 0.01 0.01
- link base_link: geometry collision cylinder length=0.05 radius=0.18; visual mesh filename=package://robotino_simulation/meshes/parts/robotino_base.dae scale=0.01 0.01 0.01
- link wheel0_link: geometry visual mesh filename=package://robotino_simulation/meshes/parts/robotino_wheel.d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 scale=0.01 0.01 0.01
- link wheel1_link: geometry visual mesh filename=package://robotino_simulation/meshes/parts/robotino_wheel.d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 scale=0.01 0.01 0.01
- link wheel2_link: geometry visual mesh filename=package://robotino_simulation/meshes/parts/robotino_wheel.d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 scale=0.01 0.01 0.01

File: robotino3_simulation/urdf/robots/robotino3_description.urdf.xacro (robot description, xacro)
@@ -6,12 +6,12 @@
   </webots>
   <!-- ros2 control include -->
-  <xacro:include filename="$(find robotino3_simulation)/urdf/robots/robotino3_ros2control.ros2_control.xacro"/>
+  <xacro:include filename="$(find robotino_simulation)/urdf/robots/robotino_ros2control.ros2_control.xacro"/>
   <!-- ros2 control instance -->
   <xacro:ros2control_wheeljoint name="WebotsControl"/>
   <!-- Instanciate and include the robotino_body -->
-  <xacro:include filename="$(find robotino3_simulation)/urdf/components/robotino_body.urdf.xacro"/>
+  <xacro:include filename="$(find robotino_simulation)/urdf/components/robotino_body.urdf.xacro"/>
   <xacro:robotino_body/>
   <!-- Instanciate and include the robotino_parts -->
-  <xacro:include filename="$(find robotino3_simulation)/urdf/components/robotino_parts.urdf.xacro"/>
+  <xacro:include filename="$(find robotino_simulation)/urdf/components/robotino_parts.urdf.xacro"/>
   <xacro:wheel name="wheel0" parent="base_link">
     <origin xyz="0.065 0.11 0.04" rpy="0 0 1.04719666667"/>
